File: rregisterA.kicad_sch (KiCad schematic)
At the start: 0 parts

Commit message: added pc, rA, rB, rI, mar
Parts:
- added D? (x8): LED, symbol Device:LED
- added R? (x8): 220, symbol Device:R
- added U? (x2): 74LS173, symbol 74xx:74LS173
- added U?: 74LS245, symbol 74xx:74LS245
Connections:
- new net: D?.1 (K), R?.1 (x8)
- new net +5V: U?.1 (A->B), U?.10 (GND), U?.16 (VCC), U?.16 (VCC)
- new net A_0: D?.2 (A), U?.6 (Q3), U?.9 (A7)
- new net A_1: D?.2 (A), U?.5 (Q2), U?.8 (A6)
- new net A_2: D?.2 (A), U?.4 (Q1), U?.7 (A5)
- new net A_3: D?.2 (A), U?.3 (Q0), U?.6 (A4)
- new net A_4: D?.2 (A), U?.5 (A3), U?.6 (Q3)
- new net A_5: D?.2 (A), U?.4 (A2), U?.5 (Q2)
- new net A_6: D?.2 (A), U?.3 (A1), U?.4 (Q1)
- new net A_7: D?.2 (A), U?.2 (A0), U?.3 (Q0)
- new net BUS_0: U?.11 (B7), U?.11 (D3)
- new net BUS_1: U?.12 (B6), U?.12 (D2)
- new net BUS_2: U?.13 (B5), U?.13 (D1)
- new net BUS_3: U?.14 (B4), U?.14 (D0)
- new net BUS_4: U?.11 (D3), U?.15 (B3)
- new net BUS_5: U?.12 (D2), U?.16 (B2)
- new net BUS_6: U?.13 (D1), U?.17 (B1)
- new net BUS_7: U?.14 (D0), U?.18 (B0)
- new net CLEAR: U?.15 (Mr), U?.15 (Mr)
- new net CLK: U?.7 (Cp), U?.7 (Cp)
- new net GND: R?.2, R?.2, R?.2, R?.2, R?.2, R?.2, R?.2, R?.2, U?.10 (E2), U?.10 (E2), U?.20 (VCC), U?.8 (GND), U?.8 (GND), U?.9 (E1), U?.9 (E1)
- new net ~{AI}: U?.1 (Oe1), U?.1 (Oe1), U?.2 (Oe2), U?.2 (Oe2)
- new net ~{AO}: U?.19 (CE)
