File: 8-bitCPU.kicad_sch (KiCad schematic)
At the start: 0 parts

Commit message: Alu & Mar
Other:
- sheet Clock ports: added CLK, HLT, ~{CLK}; removed none
- sheet Program Counter ports: added BUS_0, BUS_1, BUS_2, BUS_3, CE, CLK, CO, ~{CLR}, ~{J}; removed none
- sheet Register A: file rregisterA.kicad_sch -> registerA.kicad_sch
- sheet Register A ports: added A_0, A_1, A_2, A_3, A_4, A_5, A_6, A_7, BUS_0, BUS_1, BUS_2, BUS_3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; removed none
- sheet Register B ports: added BUS_0, BUS_1, BUS_2, BUS_3, BUS_4, BUS_5, BUS_6, BUS_7, B_0, B_1, B_2, B_3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; removed none
