File: alu.kicad_sch (KiCad schematic)
At the start: 0 parts

Commit message: Alu & Mar
Parts:
- added D? (x10): LED, symbol Device:LED
- added R? (x10): 220, symbol Device:R
- added U? (x5): 74LS02, symbol 74xx:74LS02
- added U? (x10): 74LS86, symbol 74xx:74LS86
- added U?: 74LS173, symbol 74xx:74LS173
- added U? (x4): 74LS08, symbol 74xx:74LS08
- added U? (x2): 74LS283, symbol 74xx:74LS283
- added U?: 74LS245, symbol 74xx:74LS245
Connections:
- new net: D?.1 (K), R?.1 (x10)
- new net: D?.2 (A), U?.1 (S2), U?.11, U?.8 (A6)
- new net: D?.2 (A), U?.12, U?.4 (S1), U?.9 (A7)
- new net: U?.1, U?.13
- new net: U?.11, U?.6 (B1) (x2)
- new net: U?.11 (B4), U?.3 (x2)
- new net: U?.13 (D1), U?.8
- new net: U?.1, U?.5
- new net: D?.2 (A), U?.10 (S4), U?.2, U?.2 (A0)
- new net: D?.2 (A), U?.13 (S3), U?.3, U?.3 (A1)
- new net: U?.4, U?.4
- new net: D?.2 (A), U?.1 (S2), U?.4 (A2), U?.5
- new net: D?.2 (A), U?.4 (S1), U?.5 (A3), U?.6
- new net: U?.2 (B2), U?.8 (x2)
- new net: U?.10, U?.2
- new net: D?.2 (A), U?.10 (S4), U?.6 (A4), U?.8
- new net: D?.2 (A), U?.13 (S3), U?.7 (A5), U?.9
- new net: U?.15 (B3), U?.6 (x2)
- new net: U?.10, U?.6
- new net: U?.3, U?.9
- new net: U?.7 (C0), U?.9 (C4)
- new net +5V: U?.1 (A->B), U?.14 (VCC), U?.14 (VCC), U?.14 (VCC), U?.14 (VCC), U?.16 (VCC), U?.16 (VCC), U?.16 (VCC), U?.20 (VCC)
- new net ALU_CARRY_OUT: U?.14 (D0), U?.9 (C4)
- new net A_0: U?.5 (A1)
- new net A_1: U?.3 (A2)
- new net A_2: U?.14 (A3)
- new net A_3: U?.12 (A4)
- new net A_4: U?.5 (A1)
- new net A_5: U?.3 (A2)
- new net A_6: U?.14 (A3)
- new net A_7: U?.12 (A4)
- new net BUS_0: U?.11 (B7)
- new net BUS_1: U?.12 (B6)
- new net BUS_2: U?.13 (B5)
- new net BUS_3: U?.14 (B4)
- new net BUS_4: U?.15 (B3)
- new net BUS_5: U?.16 (B2)
- new net BUS_6: U?.17 (B1)
- new net BUS_7: U?.18 (B0)
- new net B_0: U?.12
- new net B_1: U?.9
- new net B_2: U?.4
- new net B_3: U?.1
- new net B_4: U?.12
- new net B_5: U?.9
- new net B_6: U?.4
- new net B_7: U?.1
- new net CF: D?.2 (A), U?.3 (Q0)
- new net CLK: U?.7 (Cp)
- new net CLR: U?.15 (Mr)
- new net GND: R?.2, R?.2, R?.2, R?.2, R?.2, R?.2, R?.2, R?.2, R?.2, R?.2, U?.1 (Oe1), U?.10 (GND), U?.2 (Oe2), U?.7 (GND), U?.7 (GND), U?.7 (GND), U?.7 (GND), U?.8 (GND), U?.8 (GND), U?.8 (GND)
- new net SUB: U?.10, U?.10, U?.13, U?.13, U?.2, U?.2, U?.5, U?.5, U?.7 (C0)
- new net ZF: D?.2 (A), U?.4 (Q1)
- new net ~{EO}: U?.19 (CE)
- new net ~{FI}: U?.10 (E2), U?.9 (E1)
- no-connect marks 0 -> 4
