File: mar.kicad_sch (KiCad schematic)
At the start: 0 parts

Commit message: added pc, rA, rB, rI, mar
Parts:
- added D? (x4): LED, symbol Device:LED
- added R? (x4): 220, symbol Device:R
- added SW?: SW_DIP_x04, symbol Switch:SW_DIP_x04
- added U?: 74LS157, symbol 74xx:74LS157
- added U?: 74LS173, symbol 74xx:74LS173
Connections:
- new net: U?.10 (I1c), U?.4 (Q1)
- new net: U?.13 (I1d), U?.3 (Q0)
- new net: U?.3 (I1a), U?.6 (Q3)
- new net: U?.5 (Q2), U?.6 (I1b)
- new net: D?.1 (K), R?.1 (x4)
- new net BUS_0: U?.14 (D0)
- new net BUS_1: U?.13 (D1)
- new net BUS_2: U?.12 (D2)
- new net BUS_3: U?.11 (D3)
- new net GND: R?.2, R?.2, R?.2, R?.2, U?.15 (E)

Commit message: Alu & Mar
Parts:
- added D? (x2): LED, symbol Device:LED
- added J?: Conn_01x04, symbol Connector_Generic:Conn_01x04
- added R? (x2): 1k, symbol Device:R
- added SW?: SW_SPDT, symbol Switch:SW_SPDT
Connections:
- net BUS_0: now also U?.11 (D3); no longer U?.14 (D0)
- net BUS_1: now also U?.12 (D2); no longer U?.13 (D1)
- net BUS_2: now also U?.13 (D1); no longer U?.12 (D2)
- net BUS_3: now also U?.14 (D0); no longer U?.11 (D3)
- net GND: now also SW?.3, SW?.4, SW?.7, SW?.8, U?.1 (Oe1), U?.2 (Oe2), U?.8 (GND), U?.8 (GND), SW?.2 (B)
- net PROG: now reaches U?.1 (S)
- net PROG: now also D?.1 (K), SW?.1 (A)
- net at U?.10 (I1c): now also U?.5 (Q2); no longer U?.4 (Q1)
- net at U?.11 (I0c): now also SW?.2, J?.2 (Pin_2)
- net MA0: now reaches U?.12 (Zd)
- net MA0: now also D?.2 (A)
- net at U?.13 (I1d): now also U?.6 (Q3); no longer U?.3 (Q0)
- net at U?.14 (I0d): now also SW?.1, J?.1 (Pin_1)
- net +5V: now reaches U?.16 (VCC)
- net +5V: now also U?.16 (VCC), R?.1, R?.1
- net at U?.2 (I0a): now also SW?.5, J?.4 (Pin_4)
- net at U?.3 (I1a): now also U?.3 (Q0); no longer U?.6 (Q3)
- net MA3: now reaches U?.4 (Za)
- net MA3: now also D?.2 (A)
- net at U?.5 (I0b): now also SW?.6, J?.3 (Pin_3)
- net at U?.6 (I1b): now also U?.4 (Q1); no longer U?.5 (Q2)
- net MA2: now reaches U?.7 (Zb)
- net MA2: now also D?.2 (A)
- net MA1: now reaches U?.9 (Zc)
- net MA1: now also D?.2 (A)
- net ~{MI}: now reaches U?.10 (E2)
- net ~{MI}: now also U?.9 (E1)
- net CLR: now reaches U?.15 (Mr)
- net CLK: now reaches U?.7 (Cp)
- new net: D?.1 (K), SW?.3 (C)
- new net: D?.2 (A), R?.2 (x2)
Other:
- moved on the sheet: D?, R?, SW?, U?
