File: out.kicad_sch (KiCad schematic)
At the start: 0 parts

Commit message: Alu & Mar
Parts:
- added U?: AT28C16, Package_DIP:DIP-24_W15.24mm_LongPads, symbol Memory_EEPROM:AT28C16
- added U? (x4): HDSP-7403, Display_7Segment:HDSP-7401, symbol Display_Character:HDSP-7403
- added U?: 74LS08, symbol 74xx:74LS08
- added U?: 74LS273, symbol 74xx:74LS273
- added U?: LM555xN, Package_DIP:DIP-8_W7.62mm, symbol Timer:LM555xN
- added U? (x2): 74LS76, symbol 74xx:74LS76
- added U?: 74LS139, symbol 74xx:74LS139
