File: pc.kicad_sch (KiCad schematic)
At the start: 0 parts

Commit message: added pc, rA, rB, rI, mar
Parts:
- added D? (x4): LED, symbol Device:LED
- added R? (x4): 220, symbol Device:R
- added U?: 74LS245, symbol 74xx:74LS245
- added U?: 74LS161, symbol 74xx:74LS161
Connections:
- new net: D?.1 (K), R?.1 (x4)
- new net: D?.2 (A), U?.11 (Q3), U?.6 (A4)
- new net: D?.2 (A), U?.12 (Q2), U?.7 (A5)
- new net: D?.2 (A), U?.13 (Q1), U?.8 (A6)
- new net: D?.2 (A), U?.14 (Q0), U?.9 (A7)
- new net +5V: U?.16 (VCC), U?.20 (VCC)
- new net BUS_0: U?.11 (B7), U?.3 (D0)
- new net BUS_1: U?.12 (B6), U?.4 (D1)
- new net BUS_2: U?.13 (B5), U?.5 (D2)
- new net BUS_3: U?.14 (B4), U?.6 (D3)
- new net CE: U?.10 (CET), U?.7 (CEP)
- new net CLK: U?.2 (CP)
- new net CO: U?.19 (CE)
- new net GND: R?.2, R?.2, R?.2, R?.2, U?.1 (A->B), U?.10 (GND), U?.8 (GND)
- new net ~{CLEAR}: U?.1 (~{MR})
- new net ~{J}: U?.9 (~{PE})
- no-connect marks 0 -> 9
