File: registerA.kicad_sch (KiCad schematic)
At the start: 19 parts

Commit message: Alu & Mar
Parts:
- D? (x8): value LED -> (none)
- R? (x8): value 220 -> (none)
- U? (x2): value 74LS173 -> (none)
- U?: value 74LS245 -> (none)
Changed lines of the file:
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@@
       (effects (font (size 1.27 1.27)) (justify left))
     )
-    (property "Value" "220" (id 1) (at 121.92 158.115 0)
+    (property "Value" "" (id 1) (at 121.92 158.115 0)
       (effects (font (size 1.27 1.27)) (justify left))
     )
@@
       (effects (font (size 1.27 1.27)) (justify left))
     )
-    (property "Value" "220" (id 1) (at 93.98 158.115 0)
+    (property "Value" "" (id 1) (at 93.98 158.115 0)
       (effects (font (size 1.27 1.27)) (justify left))
     )
@@
       (effects (font (size 1.27 1.27)) (justify right))
     )
-    (property "Value" "LED" (id 1) (at 128.905 146.685 90)
+    (property "Value" "" (id 1) (at 128.905 146.685 90)
       (effects (font (size 1.27 1.27)) (justify right))
     )
@@
       (effects (font (size 1.27 1.27)) hide)
     )
-    (property "Value" "+5V" (id 1) (at 163.83 77.47 0))
+    (property "Value" "" (id 1) (at 163.83 77.47 0))
     (property "Footprint" "" (id 2) (at 163.83 81.915 0)
       (effects (font (size 1.27 1.27)) hide)
@@
     (in_bom yes) (on_board yes)
     (property "Reference" "U?" (id 0) (at 222.25 75.565 90))
-    (property "Value" "74LS173" (id 1) (at 225.425 93.345 90))
+    (property "Value" "" (id 1) (at 225.425 93.345 90))
     (property "Footprint" "" (id 2) (at 205.105 84.455 0)
       (effects (font (size 1.27 1.27)) hide)
@@
       (effects (font (size 1.27 1.27)) hide)
     )
-    (property "Value" "GND" (id 1) (at 52.705 88.9 0))
+    (property "Value" "" (id 1) (at 52.705 88.9 0))
     (property "Footprint" "" (id 2) (at 52.705 85.09 0)
       (effects (font (size 1.27 1.27)) hide)
@@
       (effects (font (size 1.27 1.27)) (justify right))
     )
-    (property "Value" "LED" (id 1) (at 93.98 146.685 90)
+    (property "Value" "" (id 1) (at 93.98 146.685 90)
       (effects (font (size 1.27 1.27)) (justify right))
     )
@@
       (effects (font (size 1.27 1.27)) hide)
     )
-    (property "Value" "GND" (id 1) (at 191.135 57.785 0))
+    (property "Value" "" (id 1) (at 191.135 57.785 0))
     (property "Footprint" "" (id 2) (at 191.135 53.975 0)
       (effects (font (size 1.27 1.27)) hide)
@@
       (effects (font (size 1.27 1.27)) (justify right))
     )
-    (property "Value" "LED" (id 1) (at 107.95 146.685 90)
+    (property "Value" "" (id 1) (at 107.95 146.685 90)
       (effects (font (size 1.27 1.27)) (justify right))
     )
@@
       (effects (font (size 1.27 1.27)) (justify left))
     )
-    (property "Value" "220" (id 1) (at 114.935 158.115 0)
+    (property "Value" "" (id 1) (at 114.935 158.115 0)
       (effects (font (size 1.27 1.27)) (justify left))
     )
@@
       (effects (font (size 1.27 1.27)) (justify left))
     )
-    (property "Value" "220" (id 1) (at 100.965 158.115 0)
+    (property "Value" "" (id 1) (at 100.965 158.115 0)
       (effects (font (size 1.27 1.27)) (justify left))
     )
@@
       (effects (font (size 1.27 1.27)) (justify right))
     )
-    (property "Value" "LED" (id 1) (at 86.995 146.685 90)
+    (property "Value" "" (id 1) (at 86.995 146.685 90)
       (effects (font (size 1.27 1.27)) (justify right))
     )
@@
       (effects (font (size 1.27 1.27)) (justify right))
     )
-    (property "Value" "LED" (id 1) (at 121.92 146.685 90)
+    (property "Value" "" (id 1) (at 121.92 146.685 90)
       (effects (font (size 1.27 1.27)) (justify right))
     )
@@
       (effects (font (size 1.27 1.27)) (justify left))
     )
-    (property "Value" "220" (id 1) (at 86.995 158.115 0)
+    (property "Value" "" (id 1) (at 86.995 158.115 0)
       (effects (font (size 1.27 1.27)) (justify left))
     )
@@
     (in_bom yes) (on_board yes)
     (property "Reference" "U?" (id 0) (at 156.21 74.93 90))
-    (property "Value" "74LS173" (id 1) (at 160.02 92.71 90))
+    (property "Value" "" (id 1) (at 160.02 92.71 90))
     (property "Footprint" "" (id 2) (at 139.065 83.82 0)
       (effects (font (size 1.27 1.27)) hide)
@@
       (effects (font (size 1.27 1.27)) (justify left))
     )
-    (property "Value" "220" (id 1) (at 135.89 158.115 0)
+    (property "Value" "" (id 1) (at 135.89 158.115 0)
       (effects (font (size 1.27 1.27)) (justify left))
     )
@@
       (effects (font (size 1.27 1.27)) (justify left))
     )
-    (property "Value" "220" (id 1) (at 128.905 158.115 0)
+    (property "Value" "" (id 1) (at 128.905 158.115 0)
       (effects (font (size 1.27 1.27)) (justify left))
     )
@@
       (effects (font (size 1.27 1.27)) hide)
     )
-    (property "Value" "GND" (id 1) (at 125.73 56.515 0))
+    (property "Value" "" (id 1) (at 125.73 56.515 0))
     (property "Footprint" "" (id 2) (at 125.73 52.705 0)
       (effects (font (size 1.27 1.27)) hide)
@@
       (effects (font (size 1.27 1.27)) (justify right))
     )
-    (property "Value" "LED" (id 1) (at 114.935 146.685 90)
+    (property "Value" "" (id 1) (at 114.935 146.685 90)
       (effects (font (size 1.27 1.27)) (justify right))
     )
@@
       (effects (font (size 1.27 1.27)) hide)
     )
-    (property "Value" "+5V" (id 1) (at 97.79 76.2 0))
+    (property "Value" "" (id 1) (at 97.79 76.2 0))
     (property "Footprint" "" (id 2) (at 97.79 81.915 0)
       (effects (font (size 1.27 1.27)) hide)
@@
       (effects (font (size 1.27 1.27)) hide)
     )
-    (property "Value" "+5V" (id 1) (at 229.87 78.74 0))
+    (property "Value" "" (id 1) (at 229.87 78.74 0))
     (property "Footprint" "" (id 2) (at 229.87 82.55 0)
       (effects (font (size 1.27 1.27)) hide)
@@
       (effects (font (size 1.27 1.27)) (justify right))
     )
-    (property "Value" "LED" (id 1) (at 100.965 146.685 90)
+    (property "Value" "" (id 1) (at 100.965 146.685 90)
       (effects (font (size 1.27 1.27)) (justify right))
     )
@@
     (in_bom yes) (on_board yes)
     (property "Reference" "U?" (id 0) (at 88.9 74.93 90))
-    (property "Value" "74LS245" (id 1) (at 92.075 92.71 90))
+    (property "Value" "" (id 1) (at 92.075 92.71 90))
     (property "Footprint" "" (id 2) (at 74.295 83.82 0)
       (effects (font (size 1.27 1.27)) hide)
@@
       (effects (font (size 1.27 1.27)) hide)
     )
-    (property "Value" "GND" (id 1) (at 110.49 168.275 0))
+    (property "Value" "" (id 1) (at 110.49 168.275 0))
     (property "Footprint" "" (id 2) (at 110.49 164.465 0)
       (effects (font (size 1.27 1.27)) hide)
@@
       (effects (font (size 1.27 1.27)) (justify right))
     )
-    (property "Value" "LED" (id 1) (at 135.89 146.685 90)
+    (property "Value" "" (id 1) (at 135.89 146.685 90)
       (effects (font (size 1.27 1.27)) (justify right))
     )
@@
       (effects (font (size 1.27 1.27)) hide)
     )
-    (property "Value" "GND" (id 1) (at 180.975 89.535 0))
+    (property "Value" "" (id 1) (at 180.975 89.535 0))
     (property "Footprint" "" (id 2) (at 180.975 85.725 0)
       (effects (font (size 1.27 1.27)) hide)
@@
       (effects (font (size 1.27 1.27)) (justify left))
     )
-    (property "Value" "220" (id 1) (at 107.95 158.115 0)
+    (property "Value" "" (id 1) (at 107.95 158.115 0)
       (effects (font (size 1.27 1.27)) (justify left))
     )
@@
       (effects (font (size 1.27 1.27)) hide)
     )
-    (property "Value" "GND" (id 1) (at 114.935 88.9 0))
+    (property "Value" "" (id 1) (at 114.935 88.9 0))
     (property "Footprint" "" (id 2) (at 114.935 85.09 0)
       (effects (font (size 1.27 1.27)) hide)
